Commit message: Integrate Michelo Outpost sketch launcher and add RB20 runtime support
Add an unchanged-upstream console gateway with a new-tab Sketch action, raw IPC camera bridges and fail-closed camera preflight. Include RB20-1900ES profiles, per-model calibration and the EOAT spray motion test mode. Document deployment and the remaining hardware validation prerequisites.

File: src/sketch_control/urdf/rbpodo_with_eoat.urdf.xacro (robot description, xacro)
@@ -8,5 +8,11 @@
   <xacro:arg name="cb_simulation" default="false"/>
   <xacro:arg name="model_id" default="rb10_1300e_u"/>
-  <xacro:include filename="$(find rbpodo_moveit_config)/config/rbpodo.urdf.xacro"/>
+  <xacro:property name="sketch_model_id" value="$(arg model_id)"/>
+  <xacro:if value="${sketch_model_id == 'rb20_1900es'}">
+    <xacro:include filename="rb20_sketch_arm.xacro"/>
+  </xacro:if>
+  <xacro:unless value="${sketch_model_id == 'rb20_1900es'}">
+    <xacro:include filename="$(find rbpodo_moveit_config)/config/rbpodo.urdf.xacro"/>
+  </xacro:unless>
   <xacro:include filename="$(find eoat_description)/urdf/rr_00a_b_eoat_no_camera_d405.urdf.xacro"/>
   <xacro:property name="aft200_connector_radius" value="0.005"/>
